File: ECAD/gimbal/gimbal.kicad_sch (KiCad schematic)
At the start: 15 parts, among them SW1 POWER

Commit message: Add centering and remove buttons
Parts:
- added SW2: CENTER SERVOS, Button_Switch_THT:SW_PUSH_6mm, symbol Switch:SW_Push
- added SW3: REMOVE CAMERA, Button_Switch_THT:SW_PUSH_6mm, symbol Switch:SW_Push
- C1, C2: value (none) -> 10uF; footprint (none) -> Capacitor_SMD:C_0805_2012Metric
- D1: footprint (none) -> Diode_SMD:D_SOD-123
- J2: value (none) -> UPDI; footprint (none) -> Connector_PinHeader_2.54mm:PinHeader_1x03_P2.54mm_Vertical
- J3: value (none) -> BNO1; footprint (none) -> Connector_PinHeader_2.54mm:PinHeader_1x06_P2.54mm_Vertical
- J4, J6: value (none) -> Servo; footprint (none) -> Connector_PinHeader_2.54mm:PinHeader_1x03_P2.54mm_Vertical
- J5: value (none) -> UART; footprint (none) -> Connector_PinHeader_2.54mm:PinHeader_1x02_P2.54mm_Vertical
- J7: value (none) -> BNO2; footprint (none) -> Connector_PinHeader_2.54mm:PinHeader_1x04_P2.54mm_Vertical
- R1: value (none) -> 1K; footprint (none) -> Resistor_SMD:R_1206_3216Metric
- U1: value (none) -> LM1117-3.3; footprint (none) -> Package_TO_SOT_SMD:SOT-223-3_TabPin2
- U2: value (none) -> ATtiny1604-SS; footprint (none) -> Package_SO:SOIC-14_3.9x8.7mm_P1.27mm
- gave numbers to parts that had none: 1
Connections:
- net GND: now also SW2.2, SW3.2
- net Center: now reaches U2.4 (PA6)
- net Center: now also SW2.1
- net Side: now reaches U2.5 (PA7)
- net Side: now also SW3.1

Commit message: code tuning and sch changes for v2.2
Parts:
- removed J5: UART, Connector_PinHeader_2.54mm:PinHeader_1x02_P2.54mm_Vertical, symbol Connector:Conn_01x02_Male
- added D?: POWER, symbol Device:LED
- added D?: CENTERED, symbol Device:LED
- added D?: REMOVED, symbol Device:LED
- added R? (x3): 1K, symbol Device:R
- added SW?: POWER, gimbal:Switch, symbol Switch:SW_SPDT
Connections:
- net GND: now also D?.1 (K), D?.1 (K), D?.1 (K)
- net TX: now also SW?.3 (C)
- net UPDI: now also SW?.1 (A); no longer J2.1 (Pin_1)
- net VCC: now also R?.1
- net at U2.12 (PA2): now also R?.1
- net at U2.13 (PA3): now also R?.1
- new net: J2.1 (Pin_1), SW?.2 (B)
- new net: D?.2 (A), R?.2 (x3)

Commit message: update footprints
Parts:
- D2, D3, D4: renamed from D?; footprint (none) -> Diode_SMD:D_0805_2012Metric
- R2, R3, R4: renamed from R?; footprint (none) -> Resistor_SMD:R_1206_3216Metric
- SW4: renamed from SW?; value POWER -> PRGM/DEBUG; footprint gimbal:Switch -> Button_Switch_THT:SW_Slide_1P2T_CK_OS102011MS2Q
Changed lines of the file:
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@@
   (symbol (lib_id "power:GND") (at 182.88 104.14 0) (unit 1)
     (in_bom yes) (on_board yes) (fields_autoplaced)
-    (property "Reference" "#PWR?" (id 0) (at 182.88 110.49 0)
+    (property "Reference" "#PWR0101" (id 0) (at 182.88 110.49 0)
       (effects (font (size 1.27 1.27)) hide)
     )
@@
   (symbol (lib_id "Device:LED") (at 113.03 124.46 90) (unit 1)
     (in_bom yes) (on_board yes) (fields_autoplaced)
-    (property "Reference" "D?" (id 0) (at 116.84 124.7774 90)
+    (property "Reference" "D2" (id 0) (at 116.84 124.7774 90)
       (effects (font (size 1.27 1.27)) (justify right))
     )
@@
       (effects (font (size 1.27 1.27)) (justify right))
     )
-    (property "Footprint" "" (id 2) (at 113.03 124.46 0)
+    (property "Footprint" "Diode_SMD:D_0805_2012Metric" (id 2) (at 113.03 124.46 0)
       (effects (font (size 1.27 1.27)) hide)
     )
@@
   (symbol (lib_id "Switch:SW_SPDT") (at 92.71 88.9 0) (mirror y) (unit 1)
     (in_bom yes) (on_board yes) (fields_autoplaced)
-    (property "Reference" "SW?" (id 0) (at 92.71 81.28 0))
-    (property "Value" "POWER" (id 1) (at 92.71 83.82 0))
-    (property "Footprint" "gimbal:Switch" (id 2) (at 92.71 88.9 0)
+    (property "Reference" "SW4" (id 0) (at 92.71 81.28 0))
+    (property "Value" "PRGM/DEBUG" (id 1) (at 92.71 83.82 0))
+    (property "Footprint" "Button_Switch_THT:SW_Slide_1P2T_CK_OS102011MS2Q" (id 2) (at 92.71 88.9 0)
       (effects (font (size 1.27 1.27)) hide)
     )
@@
   (symbol (lib_id "power:GND") (at 113.03 128.27 0) (unit 1)
     (in_bom yes) (on_board yes) (fields_autoplaced)
-    (property "Reference" "#PWR?" (id 0) (at 113.03 134.62 0)
+    (property "Reference" "#PWR0102" (id 0) (at 113.03 134.62 0)
       (effects (font (size 1.27 1.27)) hide)
     )
@@
   (symbol (lib_id "Device:LED") (at 175.26 97.79 90) (unit 1)
     (in_bom yes) (on_board yes) (fields_autoplaced)
-    (property "Reference" "D?" (id 0) (at 179.07 98.1074 90)
+    (property "Reference" "D3" (id 0) (at 179.07 98.1074 90)
       (effects (font (size 1.27 1.27)) (justify right))
     )
@@
       (effects (font (size 1.27 1.27)) (justify right))
     )
-    (property "Footprint" "" (id 2) (at 175.26 97.79 0)
+    (property "Footprint" "Diode_SMD:D_0805_2012Metric" (id 2) (at 175.26 97.79 0)
       (effects (font (size 1.27 1.27)) hide)
     )
@@
   (symbol (lib_id "power:VCC") (at 113.03 113.03 0) (unit 1)
     (in_bom yes) (on_board yes)
-    (property "Reference" "#PWR?" (id 0) (at 113.03 116.84 0)
+    (property "Reference" "#PWR0103" (id 0) (at 113.03 116.84 0)
       (effects (font (size 1.27 1.27)) hide)
     )
@@
   (symbol (lib_id "Device:LED") (at 190.5 97.79 90) (unit 1)
     (in_bom yes) (on_board yes) (fields_autoplaced)
-    (property "Reference" "D?" (id 0) (at 194.31 98.1074 90)
+    (property "Reference" "D4" (id 0) (at 194.31 98.1074 90)
       (effects (font (size 1.27 1.27)) (justify right))
     )
@@
       (effects (font (size 1.27 1.27)) (justify right))
     )
-    (property "Footprint" "" (id 2) (at 190.5 97.79 0)
+    (property "Footprint" "Diode_SMD:D_0805_2012Metric" (id 2) (at 190.5 97.79 0)
       (effects (font (size 1.27 1.27)) hide)
     )
@@
   (symbol (lib_id "Device:R") (at 175.26 90.17 0) (unit 1)
     (in_bom yes) (on_board yes)
-    (property "Reference" "R?" (id 0) (at 176.53 90.17 0)
+    (property "Reference" "R3" (id 0) (at 176.53 90.17 0)
       (effects (font (size 1.27 1.27)) (justify left))
     )
     (property "Value" "1K" (id 1) (at 175.26 90.17 90))
-    (property "Footprint" "" (id 2) (at 173.482 90.17 90)
+    (property "Footprint" "Resistor_SMD:R_1206_3216Metric" (id 2) (at 173.482 90.17 90)
       (effects (font (size 1.27 1.27)) hide)
     )
@@
   (symbol (lib_id "Device:R") (at 190.5 90.17 0) (unit 1)
     (in_bom yes) (on_board yes)
-    (property "Reference" "R?" (id 0) (at 191.77 90.17 0)
+    (property "Reference" "R4" (id 0) (at 191.77 90.17 0)
       (effects (font (size 1.27 1.27)) (justify left))
     )
     (property "Value" "1K" (id 1) (at 190.5 90.17 90))
-    (property "Footprint" "" (id 2) (at 188.722 90.17 90)
+    (property "Footprint" "Resistor_SMD:R_1206_3216Metric" (id 2) (at 188.722 90.17 90)
       (effects (font (size 1.27 1.27)) hide)
     )
@@
   (symbol (lib_id "Device:R") (at 113.03 116.84 0) (unit 1)
     (in_bom yes) (on_board yes)
-    (property "Reference" "R?" (id 0) (at 114.3 116.84 0)
+    (property "Reference" "R2" (id 0) (at 114.3 116.84 0)
       (effects (font (size 1.27 1.27)) (justify left))
     )
     (property "Value" "1K" (id 1) (at 113.03 116.84 90))
-    (property "Footprint" "" (id 2) (at 111.252 116.84 90)
+    (property "Footprint" "Resistor_SMD:R_1206_3216Metric" (id 2) (at 111.252 116.84 90)
       (effects (font (size 1.27 1.27)) hide)
     )
@@
     )
     (path "/074ab8fa-74e6-401f-9553-163d81a330ba"
-      (reference "#PWR?") (unit 1) (value "GND") (footprint "")
+      (reference "#PWR0101") (unit 1) (value "GND") (footprint "")
     )
     (path "/51d3a638-ca50-4002-b15d-71ceff979a8b"
-      (reference "#PWR?") (unit 1) (value "GND") (footprint "")
+      (reference "#PWR0102") (unit 1) (value "GND") (footprint "")
     )
     (path "/6f5d94a8-b089-462d-af8c-48be65890e89"
-      (reference "#PWR?") (unit 1) (value "VCC") (footprint "")
+      (reference "#PWR0103") (unit 1) (value "VCC") (footprint "")
     )
     (path "/00000000-0000-0000-0000-000061f3b730"
@@
     )
     (path "/3db22813-d923-40d6-82c8-497e87fc3e99"
-      (reference "D?") (unit 1) (value "POWER") (footprint "")
+      (reference "D2") (unit 1) (value "POWER") (footprint "Diode_SMD:D_0805_2012Metric")
     )
     (path "/6b3106cf-66f5-413e-a823-a2847d9a1f72"
-      (reference "D?") (unit 1) (value "CENTERED") (footprint "")
+      (reference "D3") (unit 1) (value "CENTERED") (footprint "Diode_SMD:D_0805_2012Metric")
     )
     (path "/bf714cbb-9dc4-4a3a-af73-58d5b3b725e1"
-      (reference "D?") (unit 1) (value "REMOVED") (footprint "")
+      (reference "D4") (unit 1) (value "REMOVED") (footprint "Diode_SMD:D_0805_2012Metric")
     )
     (path "/ed5654c2-118e-4e52-8bdd-dfce9858f506"
@@
       (reference "R1") (unit 1) (value "1K") (footprint "Resistor_SMD:R_1206_3216Metric")
     )
+    (path "/f8b4e849-5b3c-4b5a-95ce-fff91f84926b"
+      (reference "R2") (unit 1) (value "1K") (footprint "Resistor_SMD:R_1206_3216Metric")
+    )
     (path "/e07f30cd-17b8-49ab-bc1d-8fded38bd2a8"
-      (reference "R?") (unit 1) (value "1K") (footprint "")
+      (reference "R3") (unit 1) (value "1K") (footprint "Resistor_SMD:R_1206_3216Metric")
     )
     (path "/e71080b0-64cc-401b-8088-6ba190c98084"
-      (reference "R?") (unit 1) (value "1K") (footprint "")
-    )
-    (path "/f8b4e849-5b3c-4b5a-95ce-fff91f84926b"
-      (reference "R?") (unit 1) (value "1K") (footprint "")
+      (reference "R4") (unit 1) (value "1K") (footprint "Resistor_SMD:R_1206_3216Metric")
     )
     (path "/5663f4e4-1d28-460f-b8e8-94039f6b008e"
@@
     )
     (path "/43d7c944-cee7-4d2e-8279-753e3023b156"
-      (reference "SW?") (unit 1) (value "POWER") (footprint "gimbal:Switch")
+      (reference "SW4") (unit 1) (value "PRGM/DEBUG") (footprint "Button_Switch_THT:SW_Slide_1P2T_CK_OS102011MS2Q")
     )
     (path "/00000000-0000-0000-0000-000061f36cc9"
